File: hardware/kicad/esp32-emu-turbo.kicad_pcb (KiCad board)
At the start: 4 copper layers, 160 x 75 mm, 85 parts, among them J1 USB-C-16P, J3 JST-PH-2P, J4 FPC-40P-0.5mm, SW1 SW-SMD-5.1x5.1, SW10 SW-SMD-5.1x5.1, SW11 SW-SMD-5.1x5.1, SW12 SW-SMD-5.1x5.1, SW13 SW-SMD-5.1x5.1, SW2 SW-SMD-5.1x5.1, SW3 SW-SMD-5.1x5.1, SW4 SW-SMD-5.1x5.1, SW5 SW-SMD-5.1x5.1, SW6 SW-SMD-5.1x5.1, SW7 SW-SMD-5.1x5.1, SW8 SW-SMD-5.1x5.1, SW9 SW-SMD-5.1x5.1, U1 ESP32-S3-WROOM-1-N16R8, U2 ESOP-8, U3 SOT-223, U5 SOP-16, U6 TF-01A

Commit message: fix(pcb): move C1 left of AMS1117 body to fix JLCPCB component overlap
C1 (0805 input cap) was at (122, 55) — physically inside the SOT-223
body of U3 (AMS1117). JLCPCB DFM flagged component overlap.

Moved to (120, 57) — left of SOT-223 body with 2.25mm clearance,
still only 3.2mm from VIN pin for good decoupling.

All 124 tests pass (115 DFM + 9 DFA). Full release_jlcpcb sync.

Co-Authored-By: Claude Opus 4.6 (1M context) <noreply@anthropic.com>
Parts:
- moved C1 2.83 mm to (120.0, 57.0)
Routing:
- net GND: track 168.7 -> 169.2 mm
- net +5V: track 44.6 -> 44.1 mm
Changed lines of the file:
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@@
   (gr_text "C18 10uF" (at 116.0 51.5) (layer "B.Fab") (effects (font (size 0.5 0.5) (thickness 0.2)) (justify mirror)))
   (gr_text "C19 22uF" (at 110.0 61.0) (layer "B.Fab") (effects (font (size 0.5 0.5) (thickness 0.2)) (justify mirror)))
-  (gr_text "C1 10uF" (at 122.0 53.0) (layer "B.Fab") (effects (font (size 0.5 0.5) (thickness 0.2)) (justify mirror)))
+  (gr_text "C1 10uF" (at 120.0 55.0) (layer "B.Fab") (effects (font (size 0.5 0.5) (thickness 0.2)) (justify mirror)))
   (gr_text "C2 22uF" (at 125.0 60.5) (layer "B.Fab") (effects (font (size 0.5 0.5) (thickness 0.2)) (justify mirror)))
   (gr_text "L1 1uH" (at 105.5 52.5) (layer "B.Fab") (effects (font (size 0.5 0.5) (thickness 0.2)) (justify mirror)))
@@
     (pad "2" smd rect (at 0.0 0.95) (size 1.3 1.0) (layers "B.Cu" "B.Paste" "B.Mask") (net 1 "GND"))
   )
-  (footprint "C_0805" (at 122.0 55.0) (layer "B.Cu")
+  (footprint "C_0805" (at 120.0 57.0) (layer "B.Cu")
     (property "Reference" "C1" (at 0 -3 0) (layer "B.Fab") (effects (font (size 0.6 0.6) (thickness 0.2)) (justify mirror)))
     (property "Value" "C_0805" (at 0 3 0) (layer "B.Fab") (effects (font (size 0.6 0.6) (thickness 0.2)) (justify mirror)))
@@
   (segment (start 91.5 21.95) (end 91.5 23.45) (width 0.25) (layer "B.Cu") (net 1))
   (via (at 91.5 23.45) (size 0.6) (drill 0.2) (layers "F.Cu" "B.Cu") (net 1))
-  (segment (start 122.95 55.0) (end 122.95 57.5) (width 0.6) (layer "B.Cu") (net 3))
-  (via (at 122.95 57.5) (size 0.6) (drill 0.2) (layers "F.Cu" "B.Cu") (net 3))
-  (segment (start 121.05 55.0) (end 121.05 56.5) (width 0.25) (layer "B.Cu") (net 1))
-  (via (at 121.05 56.5) (size 0.6) (drill 0.2) (layers "F.Cu" "B.Cu") (net 1))
+  (segment (start 120.95 57.0) (end 120.95 59.0) (width 0.6) (layer "B.Cu") (net 3))
+  (via (at 120.95 59.0) (size 0.6) (drill 0.2) (layers "F.Cu" "B.Cu") (net 3))
+  (segment (start 119.05 57.0) (end 119.05 59.0) (width 0.25) (layer "B.Cu") (net 1))
+  (via (at 119.05 59.0) (size 0.6) (drill 0.2) (layers "F.Cu" "B.Cu") (net 1))
   (segment (start 126.5 62.5) (end 125.0 62.5) (width 0.6) (layer "B.Cu") (net 4))
   (segment (start 125.0 62.5) (end 125.0 52.35) (width 0.6) (layer "B.Cu") (net 4))
