File: hardware/kicad/06-controls.kicad_sch (KiCad schematic)
At the start: 38 parts, among them SW1 UP, SW10 SELECT, SW11 L, SW12 R, SW13 MENU, SW2 DOWN, SW3 LEFT, SW4 RIGHT, SW5 A, SW6 B, SW7 X, SW8 Y, SW9 START

Commit message: sch(layout): fix annotation overlaps across all 6 sheets — reflow to A3 where needed
Root cause: multiple sheets had annotation text boxes placed too close
to each other or to component symbols/net labels. On the live website
this rendered as strings running through each other and through
component pins — unreadable in the schematic viewer.

Per-sheet fixes:

* Sheet 1 — Power Supply
  - Upgraded to A3 landscape (was A4). USB ESD (U4/R22/R23) had
    been placed at (45, 160) directly on top of SW_PWR, C1, U3
    and C2 — all at y=160. There was no room on A4 to fit both
    the input stage (USB-C + IP5306 + battery) and the output
    stage (AMS1117 + LEDs + power switch + USB ESD) with clean
    annotations.
  - USB ESD block relocated to its own dedicated row (y=140).
  - CHARGING INDICATOR LEDs moved to a dedicated right-side zone
    (x=275, y=145) so they no longer collide with USB ESD.
  - POWER SWITCH moved to its own right-side zone (x=285, y=200)
    so its long "v1 as-built" help text no longer crosses through
    C1 / U3 (AMS1117) / C2.
  - VOLTAGE REGULATOR title + AMS1117 area pushed down (y=175 /
    y=200) with DESIGN NOTES following (y=240).
  - C18 (BAT bypass) moved left of Q1, out of the "P-MOSFET RPP /
    SI2301CDS" label zone; C27 (HF bypass) spaced further from C19
    (was 15mm gap, now 22mm) so "VOUT bulk" label no longer runs
    into "HF bypass".
  - Q1 dual annotation stacked with 3mm vertical spacing (was 2mm).
  - R24 label moved BELOW its symbol as "Q1 gate PD".
  - J3 / BT1 pushed further right (jst_x=268, bt_x=315) to use A3
    width and clear the Q1 cluster.

* Sheet 2 — MCU (ESP32-S3)
  - EN pull-up annotation shortened + moved up so it no longer
    collides with the "RC reset delay" label below.
  - BOOT switch pushed further down (c_en_y + 55) and left of the
    RESET switch so its BTN_SELECT glabel and help text no longer
    overlap the DISPLAY / AUDIO / CONTROLS annotation column. Help
    text now sits below the switch in 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
Other:
- moved on the sheet: SW13
Changed lines of the file:
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@@
   (global_label "BTN_R" (shape bidirectional) (at 363 241.81 0) (effects (font (size 1.27 1.27))) (property "Intersheetrefs" "" (at 0 0 0) (effects (font (size 1.27 1.27)) hide)))
   (wire (pts (xy 353 241.81) (xy 363 241.81)) (stroke (width 0) (type default)))
-  (text "MENU BUTTON" (at 320 235 0) (effects (font (size 2.54 2.54) bold) (justify left)))
-  (symbol (lib_id "SW_Push") (at 335 274 0) (unit 1) (exclude_from_sim no) (in_bom yes) (on_board yes) (dnp no) (property "Reference" "SW13" (at 335 269 0) (effects (font (size 1.27 1.27)))) (property "Value" "MENU" (at 335 279 0) (effects (font (size 1.27 1.27)))) (pin "1") (pin "2"))
-  (wire (pts (xy 335 258) (xy 335 274)) (stroke (width 0) (type default)))
-  (wire (pts (xy 335 274) (xy 329.92 274)) (stroke (width 0) (type default)))
-  (symbol (lib_id "GND") (at 340.08 282 0) (unit 1) (exclude_from_sim no) (in_bom no) (on_board no) (dnp no) (property "Reference" "#PWR037" (at 340.08 280 0) (effects (font (size 1.27 1.27)) hide)) (property "Value" "GND" (at 340.08 284 0) (effects (font (size 1.27 1.27)) hide)) (pin "1"))
-  (wire (pts (xy 340.08 274) (xy 340.08 282)) (stroke (width 0) (type default)))
-  (global_label "MENU_K" (shape bidirectional) (at 363 258 0) (effects (font (size 1.27 1.27))) (property "Intersheetrefs" "" (at 0 0 0) (effects (font (size 1.27 1.27)) hide)))
-  (wire (pts (xy 335 258) (xy 363 258)) (stroke (width 0) (type default)))
-  (symbol (lib_id "BAT54C") (at 375 268 0) (unit 1) (exclude_from_sim no) (in_bom yes) (on_board yes) (dnp no) (property "Reference" "D1" (at 375 263 0) (effects (font (size 1.27 1.27)))) (property "Value" "BAT54C" (at 375 273 0) (effects (font (size 1.27 1.27)))) (pin "1") (pin "2") (pin "3"))
-  (text "MENU combo" (at 378 260 0) (effects (font (size 1.5 1.5)) (justify left)))
-  (text "(START + SELECT)" (at 378 263 0) (effects (font (size 1.5 1.5)) (justify left)))
-  (global_label "MENU_K" (shape bidirectional) (at 363 268 180) (effects (font (size 1.27 1.27))) (property "Intersheetrefs" "" (at 0 0 0) (effects (font (size 1.27 1.27)) hide)))
-  (global_label "BTN_START" (shape bidirectional) (at 387 264.19 0) (effects (font (size 1.27 1.27))) (property "Intersheetrefs" "" (at 0 0 0) (effects (font (size 1.27 1.27)) hide)))
-  (global_label "BTN_SELECT" (shape bidirectional) (at 387 271.81 0) (effects (font (size 1.27 1.27))) (property "Intersheetrefs" "" (at 0 0 0) (effects (font (size 1.27 1.27)) hide)))
+  (text "MENU BUTTON" (at 115 245 0) (effects (font (size 2.54 2.54) bold) (justify left)))
+  (symbol (lib_id "SW_Push") (at 130 284 0) (unit 1) (exclude_from_sim no) (in_bom yes) (on_board yes) (dnp no) (property "Reference" "SW13" (at 130 279 0) (effects (font (size 1.27 1.27)))) (property "Value" "MENU" (at 130 289 0) (effects (font (size 1.27 1.27)))) (pin "1") (pin "2"))
+  (wire (pts (xy 130 268) (xy 130 284)) (stroke (width 0) (type default)))
+  (wire (pts (xy 130 284) (xy 124.92 284)) (stroke (width 0) (type default)))
+  (symbol (lib_id "GND") (at 135.08 292 0) (unit 1) (exclude_from_sim no) (in_bom no) (on_board no) (dnp no) (property "Reference" "#PWR037" (at 135.08 290 0) (effects (font (size 1.27 1.27)) hide)) (property "Value" "GND" (at 135.08 294 0) (effects (font (size 1.27 1.27)) hide)) (pin "1"))
+  (wire (pts (xy 135.08 284) (xy 135.08 292)) (stroke (width 0) (type default)))
+  (global_label "MENU_K" (shape bidirectional) (at 158 268 0) (effects (font (size 1.27 1.27))) (property "Intersheetrefs" "" (at 0 0 0) (effects (font (size 1.27 1.27)) hide)))
+  (wire (pts (xy 130 268) (xy 158 268)) (stroke (width 0) (type default)))
+  (symbol (lib_id "BAT54C") (at 170 278 0) (unit 1) (exclude_from_sim no) (in_bom yes) (on_board yes) (dnp no) (property "Reference" "D1" (at 170 273 0) (effects (font (size 1.27 1.27)))) (property "Value" "BAT54C" (at 170 283 0) (effects (font (size 1.27 1.27)))) (pin "1") (pin "2") (pin "3"))
+  (text "MENU combo" (at 173 270 0) (effects (font (size 1.5 1.5)) (justify left)))
+  (text "(START + SELECT)" (at 173 273 0) (effects (font (size 1.5 1.5)) (justify left)))
+  (global_label "MENU_K" (shape bidirectional) (at 158 278 180) (effects (font (size 1.27 1.27))) (property "Intersheetrefs" "" (at 0 0 0) (effects (font (size 1.27 1.27)) hide)))
+  (global_label "BTN_START" (shape bidirectional) (at 182 274.19 0) (effects (font (size 1.27 1.27))) (property "Intersheetrefs" "" (at 0 0 0) (effects (font (size 1.27 1.27)) hide)))
+  (global_label "BTN_SELECT" (shape bidirectional) (at 182 281.81 0) (effects (font (size 1.27 1.27))) (property "Intersheetrefs" "" (at 0 0 0) (effects (font (size 1.27 1.27)) hide)))
   (text "BUTTON CIRCUIT (repeated 12x):" (at 30 295 0) (effects (font (size 2.54 2.54) bold) (justify left)))
   (text "+3V3 --[10k R]-- junction --[100nF C]-- GND" (at 30 303 0) (effects (font (size 2.54 2.54)) (justify left)))
