File: hardware/kicad/06-controls.kicad_sch (KiCad schematic)
At the start: 38 parts, among them SW1 UP, SW10 SELECT, SW11 L, SW12 R, SW13 MENU, SW2 DOWN, SW3 LEFT, SW4 RIGHT, SW5 A, SW6 B, SW7 X, SW8 Y, SW9 START

Commit message: sch(fix): add missing BAT54C/USBLC6_2SC6 symbol graphics (Q1, U4, D1 were invisible)
Root cause: lib_symbols.py's SYMBOLS registry had no entries for
"BAT54C" or "USBLC6_2SC6", so lib_symbols_block() silently dropped
them. Q1 (Sheet 1), U4 (Sheet 1), and D1 (Sheet 6) existed as
Reference/Value/pin instances but had no graphic to render.

Also fixes controls.py: D1's net-label glabels were never wired to
its pins, and "BAT54C" was missing from its needed_symbols list.

ERC improved on both affected sheets (Power Supply 12->7, Controls
1->0 violations), no regressions elsewhere. DFM 119/119, DFA 9/9,
schematic<->PCB sync all pass.
Connections:
- net BTN_SELECT: now also D1.2
- net BTN_START: now also D1.1
- net MENU_K: now also D1.3
Changed lines of the file:
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@@
   (wire (pts (xy 130 268) (xy 158 268)) (stroke (width 0) (type default)))
   (symbol (lib_id "BAT54C") (at 170 278 0) (unit 1) (exclude_from_sim no) (in_bom yes) (on_board yes) (dnp no) (property "Reference" "D1" (at 170 273 0) (effects (font (size 1.27 1.27)))) (property "Value" "BAT54C" (at 170 283 0) (effects (font (size 1.27 1.27)))) (pin "1") (pin "2") (pin "3"))
-  (text "MENU combo" (at 173 270 0) (effects (font (size 1.5 1.5)) (justify left)))
-  (text "(START + SELECT)" (at 173 273 0) (effects (font (size 1.5 1.5)) (justify left)))
-  (global_label "MENU_K" (shape bidirectional) (at 158 278 180) (effects (font (size 1.27 1.27))) (property "Intersheetrefs" "" (at 0 0 0) (effects (font (size 1.27 1.27)) hide)))
-  (global_label "BTN_START" (shape bidirectional) (at 182 274.19 0) (effects (font (size 1.27 1.27))) (property "Intersheetrefs" "" (at 0 0 0) (effects (font (size 1.27 1.27)) hide)))
-  (global_label "BTN_SELECT" (shape bidirectional) (at 182 281.81 0) (effects (font (size 1.27 1.27))) (property "Intersheetrefs" "" (at 0 0 0) (effects (font (size 1.27 1.27)) hide)))
+  (text "MENU combo" (at 182 274 0) (effects (font (size 1.5 1.5)) (justify left)))
+  (text "(START + SELECT)" (at 182 277 0) (effects (font (size 1.5 1.5)) (justify left)))
+  (global_label "MENU_K" (shape bidirectional) (at 170 268 90) (effects (font (size 1.27 1.27))) (property "Intersheetrefs" "" (at 0 0 0) (effects (font (size 1.27 1.27)) hide)))
+  (wire (pts (xy 170 273) (xy 170 268)) (stroke (width 0) (type default)))
+  (global_label "BTN_START" (shape bidirectional) (at 159 279.27 180) (effects (font (size 1.27 1.27))) (property "Intersheetrefs" "" (at 0 0 0) (effects (font (size 1.27 1.27)) hide)))
+  (wire (pts (xy 165 279.27) (xy 159 279.27)) (stroke (width 0) (type default)))
+  (global_label "BTN_SELECT" (shape bidirectional) (at 181 279.27 0) (effects (font (size 1.27 1.27))) (property "Intersheetrefs" "" (at 0 0 0) (effects (font (size 1.27 1.27)) hide)))
+  (wire (pts (xy 175 279.27) (xy 181 279.27)) (stroke (width 0) (type default)))
   (text "BUTTON CIRCUIT (repeated 12x):" (at 30 295 0) (effects (font (size 2.54 2.54) bold) (justify left)))
   (text "+3V3 --[10k R]-- junction --[100nF C]-- GND" (at 30 303 0) (effects (font (size 2.54 2.54)) (justify left)))
