File: hardware/kicad/06-controls.kicad_sch (KiCad schematic)
At the start: 38 parts, among them SW1 UP, SW10 SELECT, SW11 L, SW12 R, SW13 MENU, SW2 DOWN, SW3 LEFT, SW4 RIGHT, SW5 A, SW6 B, SW7 X, SW8 Y, SW9 START

Commit message: sch+tools: fix schematic/PCB pin divergence, recalibrate USB check to Full Speed, make verify-all mean "all"
Failure 1 — verify_netlist_diff T4 (4 mismatches + 2 suppression mechanisms)

Schematic side was wrong in every case; decided from datasheets, not convenience.

* U4 (USBLC6-2SC6, ST doc ID 11265 Rev 5): pins 1/6 are one internal
  I/O node and pins 3/4 the other. The schematic had USB_DM_MCU on
  pin 6 and USB_DP_MCU on pin 4, which shorts R23/R22 out inside the
  package. Both pins of each pair now sit on the connector-side net,
  matching routing.py and hardware/datasheet_specs.py.
* U4 pin 5 is the VBUS clamp reference; the schematic tied it to +5V,
  the IP5306 boost OUTPUT, which is live with no cable attached. Now
  VBUS, as the board already had it.
* U3 (AMS1117): the library symbol used the generic 1=VIN/2=GND/3=VOUT
  numbering. The SOT-223 datasheet land is 1=GND/2=VOUT/3=VIN plus a
  tab (4) that is VOUT. Symbol renumbered, tab pin added; drawing
  unchanged.
* C24/C27/C21 and the twelve button pull-ups R4..R15 had pin 1 and
  pin 2 the opposite way round from their footprints. Symbol
  placement now supports a rotation angle, and these symmetric
  two-terminal parts are placed at 180 deg so the pin numbers agree
  with the pads without altering how the sheet looks.

Real schematic defects found while doing the above:

* Sheets 4 and 5 dropped a GND stub straight through the anchor of the
  label below it: SD_CS was shorted to GND on the SD sheet and the
  PAM8403 audio input was shorted to GND on the audio sheet.
* R22 and R23 were wired with horizontal stubs against a symbol whose
  pins are vertical, so both series termination resistors were
  completely floating in the exported netlist.
* Same class: C22 (the audio DC-block) and the top terminals of
  R20/R21 were attached to nothing.
* The display sheet walked the FPC symbol pins backwards and ran one
  step off the end, so LCD_D7 never reached J4 — the schematic showed
  a 7-bit data bus. I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
Connections:
- net BTN_A: now also R8.1; no longer R8.2
- net BTN_B: now also R9.1; no longer R9.2
- net BTN_DOWN: now also R5.1; no longer R5.2
- net BTN_L: now also R14.1; no longer R14.2
- net BTN_LEFT: now also R6.1; no longer R6.2
- net BTN_R: now also R15.1; no longer R15.2
- net BTN_RIGHT: now also R7.1; no longer R7.2
- net BTN_SELECT: now also R13.1; no longer R13.2
- net BTN_START: now also R12.1; no longer R12.2
- net BTN_UP: now also R4.1; no longer R4.2
- net BTN_X: now also R10.1; no longer R10.2
- net BTN_Y: now also R11.1; no longer R11.2
Other:
- moved on the sheet: R10, R11, R12, R13, R14, R15, R4, R5, R6, R7, R8, R9
