File: hardware/kicad/01-power-supply.kicad_sch (KiCad schematic)
At the start: 25 parts, among them J1 USB_C, J3 JST PH 2-pin, Q1 SI2301CDS, U2 IP5306, U3 AMS1117-3.3, U4 USBLC6-2SC6

Commit message: sch(fix): add missing BAT54C/USBLC6_2SC6 symbol graphics (Q1, U4, D1 were invisible)
Root cause: lib_symbols.py's SYMBOLS registry had no entries for
"BAT54C" or "USBLC6_2SC6", so lib_symbols_block() silently dropped
them. Q1 (Sheet 1), U4 (Sheet 1), and D1 (Sheet 6) existed as
Reference/Value/pin instances but had no graphic to render.

Also fixes controls.py: D1's net-label glabels were never wired to
its pins, and "BAT54C" was missing from its needed_symbols list.

ERC improved on both affected sheets (Power Supply 12->7, Controls
1->0 violations), no regressions elsewhere. DFM 119/119, DFA 9/9,
schematic<->PCB sync all pass.
Connections:
- net +5V: now also U4.5 (VBUS)
- net USB_D+: now also U4.3 (I/O2_A)
- net USB_D-: now also U4.1 (I/O1_A)
- net USB_DM_MCU: now also U4.6 (I/O1_B)
- net USB_DP_MCU: now also U4.4 (I/O2_B)
- net at C18.1, L1.2, U2.6 (BAT): now also Q1.3
- net at J3.1 (+), J3.2 (-): now also Q1.2
- net at R24.1: now also Q1.1
