File: hardware/kicad/03-display.kicad_sch (KiCad schematic)
At the start: 2 parts, among them J4 FPC-16P-0.5mm, U4 ILI9488 4.0in 8080

Commit message: fix(hw): R4 audit — schematic↔PCB sync guard + 4 fixes + R4-CRIT-1 false-positive closure
Round 4 of the hardware audit found four real schematic/PCB drift bugs
that rounds 1-3 missed because no check cross-validated the two Python
generators. A fifth finding (R4-CRIT-1, "FPC pinout mismatch") turned
out to be a FALSE POSITIVE caused by the landscape FPC pin reversal
(connector_pad = 41 − panel_pin) — verified programmatically against
all 40 J4 pads of the panel datasheet in components.md.

Fixes applied:
  R4-HIGH-1  USBLC6 (U4) + R22/R23 instantiated in power_supply.py —
             previously only in routing.py, invisible to schematic
             review.
  R4-HIGH-2  Display module symbol ref renamed U4 → DS1 in display.py.
             U4 is now cleanly owned by the physical USBLC6 TVS.
  R4-HIGH-3  PAM8403 R20/R21 input bias moved from GND to VREF
             (pin 8) per the datasheet single-ended app circuit.
  R4-CRIT-1  CLOSED as false positive. Both display.py (panel-side)
             and datasheet_specs.py (connector-side) were correct all
             along. Added 41-N reversal documentation at the top of
             both files so the mistake can't be re-raised.
  ERC CRIT   Pre-existing "Power output ↔ Power output" on +5V was
             PWR_FLAG duplicating IP5306 VOUT (already power_out in the
             library symbol). Removed the PWR_FLAG. ERC now 0 critical.

Incidental cleanups required by the new sync guard:
  - mcu.py R3 (external EN pull-up) removed from schematic — already
    DNP in BOM because the WROOM-1 module has an internal pull-up.
  - controls.py D1 BAT54C (MENU combo diode) instantiated in schematic
    to match the PCB routing. MENU button wiring simplified to the
    MENU_K node; there is no dedicated BTN_MENU GPIO (firmware detects
    START+SELECT combo).
  - power_supply.py USB_CC1 / USB_CC2 global labels added so the
    connector-net coverage check sees the full USB-C net set.
  - display.py docstring expanded with the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
Parts:
- renumbered U4 to DS1
Other:
- note added: "ILI9488 Panel FPC-40P Pin Mapping (source: components.md):"
- note added: "Panel 17-24=DB0-DB7 33=LED-A(BL) 34-36=LED-K(GND) 38,39=IM0,IM1(+3V3) 40=IM2(GND)"
- note added: "Panel 6,7=VDDI/VDDA(+3V3) 9=CS 10=DC 11=WR 12=RD 15=RESET"
- note added: "e.g. panel pin 17 (DB0) contacts J4 pad 24. See datasheet_specs.py for the connector-side mapping."
- note added: "⚠ FPC PIN REVERSAL on PCB: panel pin N ↔ J4 pad (41-N)."
- note removed: "- No level shifter: ESP32-S3 GPIO = 3.3V = display logic level"
- note removed: "FPC 17-24=DB0-DB7 33=LED-A(BL) 34-36=LED-K(GND) 38,39=IM0,IM1(+3V3) 40=IM2(GND)"
- note removed: "FPC 6,7=VDDI/VDDA(+3V3) 9=CS 10=DC 11=WR 12=RD 15=RESET"
- note removed: "ILI9488 FPC-40P Pin Mapping:"
Changed lines of the file:
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@@
   (text "DISPLAY - ILI9488 4.0in 320x480" (at 30 25 0) (effects (font (size 5 5) bold) (justify left)))
   (text "8-bit 8080 parallel interface (mandatory for SNES emulation speed)" (at 30 33 0) (effects (font (size 2.54 2.54)) (justify left)))
-  (symbol (lib_id "ST7796S_Module") (at 148 120 0) (unit 1) (exclude_from_sim no) (in_bom yes) (on_board yes) (dnp no) (property "Reference" "U4" (at 148 115 0) (effects (font (size 1.27 1.27)))) (property "Value" "ILI9488 4.0in 8080" (at 148 125 0) (effects (font (size 1.27 1.27)))) (pin "1") (pin "2") (pin "3") (pin "4") (pin "5") (pin "6") (pin "7") (pin "8") (pin "9") (pin "10") (pin "11") (pin "12") (pin "13") (pin "14") (pin "15") (pin "16"))
+  (symbol (lib_id "ST7796S_Module") (at 148 120 0) (unit 1) (exclude_from_sim no) (in_bom yes) (on_board yes) (dnp no) (property "Reference" "DS1" (at 148 115 0) (effects (font (size 1.27 1.27)))) (property "Value" "ILI9488 4.0in 8080" (at 148 125 0) (effects (font (size 1.27 1.27)))) (pin "1") (pin "2") (pin "3") (pin "4") (pin "5") (pin "6") (pin "7") (pin "8") (pin "9") (pin "10") (pin "11") (pin "12") (pin "13") (pin "14") (pin "15") (pin "16"))
   (global_label "+3V3" (shape input) (at 118 104.76 0) (effects (font (size 1.27 1.27))) (property "Intersheetrefs" "" (at 0 0 0) (effects (font (size 1.27 1.27)) hide)))
   (wire (pts (xy 118 104.76) (xy 137.84 104.76)) (stroke (width 0) (type default)))
@@
   (global_label "LCD_D7" (shape input) (at 242.38 99.68 180) (effects (font (size 1.27 1.27))) (property "Intersheetrefs" "" (at 0 0 0) (effects (font (size 1.27 1.27)) hide)))
   (wire (pts (xy 252.38 99.68) (xy 242.38 99.68)) (stroke (width 0) (type default)))
-  (text "ILI9488 FPC-40P Pin Mapping:" (at 30 180 0) (effects (font (size 2.54 2.54) bold) (justify left)))
-  (text "FPC 6,7=VDDI/VDDA(+3V3)  9=CS  10=DC  11=WR  12=RD  15=RESET" (at 30 188 0) (effects (font (size 2.54 2.54)) (justify left)))
-  (text "FPC 17-24=DB0-DB7  33=LED-A(BL)  34-36=LED-K(GND)  38,39=IM0,IM1(+3V3)  40=IM2(GND)" (at 30 194 0) (effects (font (size 2.54 2.54)) (justify left)))
+  (text "ILI9488 Panel FPC-40P Pin Mapping (source: components.md):" (at 30 180 0) (effects (font (size 2.54 2.54) bold) (justify left)))
+  (text "Panel 6,7=VDDI/VDDA(+3V3)  9=CS  10=DC  11=WR  12=RD  15=RESET" (at 30 188 0) (effects (font (size 2.54 2.54)) (justify left)))
+  (text "Panel 17-24=DB0-DB7  33=LED-A(BL)  34-36=LED-K(GND)  38,39=IM0,IM1(+3V3)  40=IM2(GND)" (at 30 194 0) (effects (font (size 2.54 2.54)) (justify left)))
   (text "Interface mode: IM2=0 IM1=1 IM0=1 = 8080 8-bit parallel" (at 30 200 0) (effects (font (size 2.54 2.54)) (justify left)))
   (text "- GPIO4-11 form contiguous 8-bit bus for efficient register-level DMA" (at 30 208 0) (effects (font (size 2.54 2.54)) (justify left)))
   (text "- WR strobes data on rising edge, RD tied HIGH (+3V3, write-only mode)" (at 30 214 0) (effects (font (size 2.54 2.54)) (justify left)))
-  (text "- No level shifter: ESP32-S3 GPIO = 3.3V = display logic level" (at 30 220 0) (effects (font (size 2.54 2.54)) (justify left)))
+  (text "⚠ FPC PIN REVERSAL on PCB: panel pin N ↔ J4 pad (41-N)." (at 30 222 0) (effects (font (size 2.54 2.54)) (justify left)))
+  (text "  e.g. panel pin 17 (DB0) contacts J4 pad 24. See datasheet_specs.py for the connector-side mapping." (at 30 228 0) (effects (font (size 2.54 2.54)) (justify left)))
   (sheet_instances (path "/" (page "3")))
 )

Commit message: sch(layout): fix annotation overlaps across all 6 sheets — reflow to A3 where needed
Root cause: multiple sheets had annotation text boxes placed too close
to each other or to component symbols/net labels. On the live website
this rendered as strings running through each other and through
component pins — unreadable in the schematic viewer.

Per-sheet fixes:

* Sheet 1 — Power Supply
  - Upgraded to A3 landscape (was A4). USB ESD (U4/R22/R23) had
    been placed at (45, 160) directly on top of SW_PWR, C1, U3
    and C2 — all at y=160. There was no room on A4 to fit both
    the input stage (USB-C + IP5306 + battery) and the output
    stage (AMS1117 + LEDs + power switch + USB ESD) with clean
    annotations.
  - USB ESD block relocated to its own dedicated row (y=140).
  - CHARGING INDICATOR LEDs moved to a dedicated right-side zone
    (x=275, y=145) so they no longer collide with USB ESD.
  - POWER SWITCH moved to its own right-side zone (x=285, y=200)
    so its long "v1 as-built" help text no longer crosses through
    C1 / U3 (AMS1117) / C2.
  - VOLTAGE REGULATOR title + AMS1117 area pushed down (y=175 /
    y=200) with DESIGN NOTES following (y=240).
  - C18 (BAT bypass) moved left of Q1, out of the "P-MOSFET RPP /
    SI2301CDS" label zone; C27 (HF bypass) spaced further from C19
    (was 15mm gap, now 22mm) so "VOUT bulk" label no longer runs
    into "HF bypass".
  - Q1 dual annotation stacked with 3mm vertical spacing (was 2mm).
  - R24 label moved BELOW its symbol as "Q1 gate PD".
  - J3 / BT1 pushed further right (jst_x=268, bt_x=315) to use A3
    width and clear the Q1 cluster.

* Sheet 2 — MCU (ESP32-S3)
  - EN pull-up annotation shortened + moved up so it no longer
    collides with the "RC reset delay" label below.
  - BOOT switch pushed further down (c_en_y + 55) and left of the
    RESET switch so its BTN_SELECT glabel and help text no longer
    overlap the DISPLAY / AUDIO / CONTROLS annotation column. Help
    text now sits below the switch in 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
Other:
- note added: "+3V3 (FPC12, RO)"
- note added: "+3V3 (FPC33, BL)"
- note added: "GPIO12 / FPC9"
- note added: "GPIO13 / FPC15"
- note added: "GPIO14 / FPC10"
- note added: "GPIO46 / FPC11"
- note removed: "+3V3 tied (FPC12, write-only)"
- note removed: "+3V3 tied (FPC33, always-on)"
- note removed: "GPIO12 (FPC9)"
- note removed: "GPIO13 (FPC15)"
- note removed: "GPIO14 (FPC10)"
- note removed: "GPIO46 (FPC11)"
Changed lines of the file:
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@@
   (symbol (lib_id "GND") (at 118 107.3 0) (unit 1) (exclude_from_sim no) (in_bom no) (on_board no) (dnp no) (property "Reference" "#PWR001" (at 118 105.3 0) (effects (font (size 1.27 1.27)) hide)) (property "Value" "GND" (at 118 109.3 0) (effects (font (size 1.27 1.27)) hide)) (pin "1"))
   (wire (pts (xy 118 107.3) (xy 137.84 107.3)) (stroke (width 0) (type default)))
-  (text "Control signals:" (at 88 106 0) (effects (font (size 2 2) bold) (justify left)))
+  (text "Control signals:" (at 76 106 0) (effects (font (size 2 2) bold) (justify left)))
   (wire (pts (xy 137.84 109.84) (xy 112.84 109.84)) (stroke (width 0) (type default)))
   (global_label "LCD_CS" (shape bidirectional) (at 112.84 109.84 180) (effects (font (size 1.27 1.27))) (property "Intersheetrefs" "" (at 0 0 0) (effects (font (size 1.27 1.27)) hide)))
-  (text "GPIO12 (FPC9)" (at 87.84 109.84 0) (effects (font (size 1.5 1.5)) (justify left)))
+  (text "GPIO12 / FPC9" (at 75.84 109.84 0) (effects (font (size 1.5 1.5)) (justify left)))
   (wire (pts (xy 137.84 112.38) (xy 112.84 112.38)) (stroke (width 0) (type default)))
   (global_label "LCD_RST" (shape bidirectional) (at 112.84 112.38 180) (effects (font (size 1.27 1.27))) (property "Intersheetrefs" "" (at 0 0 0) (effects (font (size 1.27 1.27)) hide)))
-  (text "GPIO13 (FPC15)" (at 87.84 112.38 0) (effects (font (size 1.5 1.5)) (justify left)))
+  (text "GPIO13 / FPC15" (at 75.84 112.38 0) (effects (font (size 1.5 1.5)) (justify left)))
   (wire (pts (xy 137.84 114.92) (xy 112.84 114.92)) (stroke (width 0) (type default)))
   (global_label "LCD_DC" (shape bidirectional) (at 112.84 114.92 180) (effects (font (size 1.27 1.27))) (property "Intersheetrefs" "" (at 0 0 0) (effects (font (size 1.27 1.27)) hide)))
-  (text "GPIO14 (FPC10)" (at 87.84 114.92 0) (effects (font (size 1.5 1.5)) (justify left)))
+  (text "GPIO14 / FPC10" (at 75.84 114.92 0) (effects (font (size 1.5 1.5)) (justify left)))
   (wire (pts (xy 137.84 117.46) (xy 112.84 117.46)) (stroke (width 0) (type default)))
   (global_label "LCD_WR" (shape bidirectional) (at 112.84 117.46 180) (effects (font (size 1.27 1.27))) (property "Intersheetrefs" "" (at 0 0 0) (effects (font (size 1.27 1.27)) hide)))
-  (text "GPIO46 (FPC11)" (at 87.84 117.46 0) (effects (font (size 1.5 1.5)) (justify left)))
+  (text "GPIO46 / FPC11" (at 75.84 117.46 0) (effects (font (size 1.5 1.5)) (justify left)))
   (wire (pts (xy 137.84 120) (xy 112.84 120)) (stroke (width 0) (type default)))
   (global_label "LCD_RD" (shape bidirectional) (at 112.84 120 180) (effects (font (size 1.27 1.27))) (property "Intersheetrefs" "" (at 0 0 0) (effects (font (size 1.27 1.27)) hide)))
-  (text "+3V3 tied (FPC12, write-only)" (at 87.84 120 0) (effects (font (size 1.5 1.5)) (justify left)))
+  (text "+3V3 (FPC12, RO)" (at 75.84 120 0) (effects (font (size 1.5 1.5)) (justify left)))
   (wire (pts (xy 137.84 125.08) (xy 112.84 125.08)) (stroke (width 0) (type default)))
   (global_label "LCD_BL" (shape bidirectional) (at 112.84 125.08 180) (effects (font (size 1.27 1.27))) (property "Intersheetrefs" "" (at 0 0 0) (effects (font (size 1.27 1.27)) hide)))
-  (text "+3V3 tied (FPC33, always-on)" (at 87.84 125.08 0) (effects (font (size 1.5 1.5)) (justify left)))
+  (text "+3V3 (FPC33, BL)" (at 75.84 125.08 0) (effects (font (size 1.5 1.5)) (justify left)))
   (text "8-bit data bus:" (at 173 100 0) (effects (font (size 2 2) bold) (justify left)))
   (wire (pts (xy 158.16 104.76) (xy 183.16 104.76)) (stroke (width 0) (type default)))
